Commit message: Update deliver_rb_new.urdf.xacro

File: urdf/deliver_rb_new.urdf.xacro (robot description, xacro)
@@ -82,5 +82,5 @@
       <geometry>
         <mesh
-          filename="package://fix/meshes/base_link.STL" />
+          filename="package://deliver_rb/meshes/base_link.STL" />
       </geometry>
       <material
@@ -96,5 +96,5 @@
       <geometry>
         <mesh
-          filename="package://fix/meshes/base_link.STL" />
+          filename="package://deliver_rb/meshes/base_link.STL" />
       </geometry>
     </collision>
@@ -122,5 +122,5 @@
       <geometry>
         <mesh
-          filename="package://fix/meshes/right_wheel.STL" />
+          filename="package://deliver_rb/meshes/right_wheel.STL" />
       </geometry>
       <material
@@ -136,5 +136,5 @@
       <geometry>
         <mesh
-          filename="package://fix/meshes/right_wheel.STL" />
+          filename="package://deliver_rb/meshes/right_wheel.STL" />
       </geometry>
     </collision>
@@ -175,5 +175,5 @@
       <geometry>
         <mesh
-          filename="package://fix/meshes/left_wheel.STL" />
+          filename="package://deliver_rb/meshes/left_wheel.STL" />
       </geometry>
       <material
@@ -189,5 +189,5 @@
       <geometry>
         <mesh
-          filename="package://fix/meshes/left_wheel.STL" />
+          filename="package://deliver_rb/meshes/left_wheel.STL" />
       </geometry>
     </collision>
@@ -228,5 +228,5 @@
       <geometry>
         <mesh
-          filename="package://fix/meshes/pole.STL" />
+          filename="package://deliver_rb/meshes/pole.STL" />
       </geometry>
       <material
@@ -242,5 +242,5 @@
       <geometry>
         <mesh
-          filename="package://fix/meshes/pole.STL" />
+          filename="package://deliver_rb/meshes/pole.STL" />
       </geometry>
     </collision>
@@ -281,5 +281,5 @@
       <geometry>
         <mesh
-          filename="package://fix/meshes/free_forward.STL" />
+          filename="package://deliver_rb/meshes/free_forward.STL" />
       </geometry>
       <material
@@ -295,5 +295,5 @@
       <geometry>
         <mesh
-          filename="package://fix/meshes/free_forward.STL" />
+          filename="package://deliver_rb/meshes/free_forward.STL" />
       </geometry>
     </collision>
@@ -334,5 +334,5 @@
       <geometry>
         <mesh
-          filename="package://fix/meshes/free_backward.STL" />
+          filename="package://deliver_rb/meshes/free_backward.STL" />
       </geometry>
       <material
@@ -348,5 +348,5 @@
       <geometry>
         <mesh
-          filename="package://fix/meshes/free_backward.STL" />
+          filename="package://deliver_rb/meshes/free_backward.STL" />
       </geometry>
     </collision>
@@ -387,5 +387,5 @@
       <geometry>
         <mesh
-          filename="package://fix/meshes/basket.STL" />
+          filename="package://deliver_rb/meshes/basket.STL" />
       </geometry>
       <material
@@ -401,5 +401,5 @@
       <geometry>
         <mesh
-          filename="package://fix/meshes/basket.STL" />
+          filename="package://deliver_rb/meshes/basket.STL" />
       </geometry>
     </collision>
@@ -440,5 +440,5 @@
       <geometry>
         <mesh
-          filename="package://fix/meshes/hat.STL" />
+          filename="package://deliver_rb/meshes/hat.STL" />
       </geometry>
       <material
@@ -454,5 +454,5 @@
       <geometry>
         <mesh
-          filename="package://fix/meshes/hat.STL" />
+          filename="package://deliver_rb/meshes/hat.STL" />
       </geometry>
     </collision>
@@ -471,30 +471,3 @@
       xyz="0 0 0" />
   </joint>
-  <!-- Hokuyo Laser -->
-  <!-- <link name="laser">
-    <collision>
-      <origin xyz="0 0 0" rpy="0 0 0"/>
-      <geometry>
-    <box size="0.1 0.1 0.1"/>
-      </geometry>
-    </collision>
-    <visual>
-      <origin xyz="0.0 0 0" rpy="0 0 0"/>
-      <geometry>
-        <mesh filename="package://deliver_rb/meshes/hokuyo.dae"/>
-      </geometry>
-    </visual>
-    <inertial>
-      <mass value="1e-5" />
-      <origin xyz="0 0 0" rpy="0 0 0"/>
-      <inertia ixx="1e-6" ixy="0" ixz="0" iyy="1e-6" iyz="0" izz="1e-6" />
-    </inertial>
-  </link> -->
-  <!-- CPU Lidar join-->
-  <!-- <joint name="laser_join" type="fixed">
-    <axis xyz="0 0 0" />
-    <origin xyz="0 0.2 0.04" rpy="0 0 0"/>
-    <parent link="base_link"/>
-    <child link="laser"/>
-  </joint> -->
 </robot>
